File: HidroProject.kicad_pcb (KiCad board)
At the start: 4 copper layers, 110 x 60.5 mm, 121 parts, among them IC1 DALC208SC6, J1 691322310002, J11 67996-412HLF, J2 691322310002, J3 691322310002, J4 SM03B-SRSS-TB, J5 JAE_SIM_Card_SF72S006, J6 U.FL-R-SMT-1_10_, J7 691322310002, J8 USB_C_Receptacle_USB2.0_16P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

Commit message: mahlas guncellendi
Other:
- board text added: "OES"
- board text removed: "O.E."
